File: KiCAD/Line_Follower.kicad_sch (KiCad schematic)
At the start: 4 parts

Commit message: Updated schematics and design
Parts:
- added U7: BOB-12009, CONV_BOB-12009, symbol BOB-12009:BOB-12009
- gave numbers to parts that had none: 4
Connections:
- net 5V: now also U7.HV
- net GND: now also U7.GND_1 (GND), U7.GND_2 (GND)
- net Motor Driver/D10/PWM: now also U7.HV4; no longer U1.28 (D10/PWM)
- net Motor Driver/D5/PWM: now also U7.HV1; no longer U1.23 (D5/PWM)
- net Motor Driver/D6/PWM: now also U7.HV2; no longer U1.24 (D6/PWM)
- net Motor Driver/D9/PWM: now also U7.HV3; no longer U1.27 (D9/PWM)
- net Motor Driver/D4: now reaches U2.HV3
- net at U1.2 (+3V3), U2.LV: now also U7.LV
- net at U2.LV3: now also U1.22 (D4)
- net Motor Driver/D8: no longer names the net of U1.26 (D8)
- new net: U1.23 (D5/PWM), U7.LV1
- new net: U1.24 (D6/PWM), U7.LV2
- new net: U1.27 (D9/PWM), U7.LV3
- new net: U1.28 (D10/PWM), U7.LV4
Other:
- sheet Motor Driver ports: added D4; removed D8
- note removed: "06.08.2023"
- note removed: "Friso Vijverberg Liam Breytenbach Julian Dower University of Cape Town EEE3099S"
- note removed: "Line Following Robot Schematic"
- note removed: "Line Sensors Complete Motot LED"
- note removed: "Not sure if I've done the power symbols right. Double check"
- note removed: "v 1.0"
- title: (none) -> Line Following Robot Schematic
- moved on the sheet: U3

Commit message: Add files via upload
Parts:
- added R6: 220, symbol Device:R
- U1: value ABX00027 -> Arduino
- U2: value BOB-12009 -> LVL Shifter
- U3: renamed from U7; value BOB-12009 -> LVL Shifter
- U7: renamed from U3; value HC-SR04 -> Ultrasonic
Connections:
- net SEN0 is gone; now on net SEN1: U1.4 (A0/DAC0)
- net SEN1: no longer U1.5 (A1)
- net SEN2: now also U1.5 (A1); no longer U1.6 (A2)
- net SEN3: now also U1.6 (A2); no longer U1.7 (A3)
- net at D1.2 (A): now also R6.1; no longer U1.11 (A7)
- net +3V3: now reaches U1.2 (+3V3), U2.LV, U3.LV
- net D5: now reaches U3.LV1
- net D5: no longer U1.23 (D5/PWM)
- net D6: now reaches U3.LV2
- net D6: no longer U1.24 (D6/PWM)
- net D9: now reaches U3.LV3
- net D9: no longer U1.27 (D9/PWM)
- net D10: now reaches U3.LV4
- net D10: no longer U1.28 (D10/PWM)
- net TRIG: now reaches U2.HV1
- net TRIG: no longer U7.2 (TRIG)
- net ECHO: now reaches U2.HV2
- net ECHO: no longer U7.3 (ECHO)
- net D2: now reaches U2.LV1
- net D2: no longer U1.20 (D2)
- net D3: now reaches U2.LV2
- net D3: no longer U1.21 (D3/PWM)
- net D4: now reaches U2.LV3
- net D4: no longer U1.22 (D4)
- net 5V renamed +5V
- net Motor Driver/D10/PWM renamed IN4
- net Motor Driver/D4 renamed EN
- net Motor Driver/D5/PWM renamed IN1
- net Motor Driver/D6/PWM renamed IN2
- net Motor Driver/D9/PWM renamed IN3
- new net: R6.2, U1.11 (A7)
- new net SEN4: U1.7 (A3)
- new net U2_HV1: U7.2 (TRIG)
- new net U2_HV2: U7.3 (ECHO)
- new net U2_LV1: U1.20 (D2)
- new net U2_LV2: U1.21 (D3/PWM)
- new net U2_LV3: U1.22 (D4)
- new net U3_LV1: U1.23 (D5/PWM)
- new net U3_LV2: U1.24 (D6/PWM)
- new net U3_LV3: U1.27 (D9/PWM)
- new net U3_LV4: U1.28 (D10/PWM)
- no-connect marks 0 -> 15
Other:
- sheet Line_Tracking ports: added GND, SEN, Vcc; removed none
- sheet Motor Driver ports: added EN, IN1, IN2, IN3, IN4; removed D10/PWM, D4, D5/PWM, D6/PWM, D9/PWM
- note added: "Electro-mechanical Subsystem"
- note added: "Level Shifters"
- note added: "Line Tracking Sensor"
- note added: "Microcontroller Subsystem"
- note added: "Ultrasonic Sensor"
- note removed: "Add 5th sensor?"
- moved on the sheet: D1, U1, U2, U3, U7
