File: KiCAD/Line_Follower_Top_Right.kicad_pcb (KiCad board)
At the start: 2 copper layers, 50 x 100 mm, 3 parts

Commit message: Add files via upload
Other:
- board size 50 x 100 mm -> 407.7 x 189.3 mm
- board text added: "Line Sensors (SEN)"
- board text added: "Ultrasonic Sensor"
Changed lines of the file:
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@@
     (pad "LV4" thru_hole circle locked (at -5.08 6.35 90) (size 1.524 1.524) (drill 1.016) (layers *.Cu *.Mask))
   )
-  (gr_circle (center 101.46 157.34) (end 186.46 157.34) (layer "Dwgs.User") (width 0.2) (fill none))
+  (gr_rect (start 424.18 33.02) (end 426.72 48.26) (layer "F.Adhes") (width 0.05) (fill none))
+  (gr_rect (start 424.18 53.34) (end 421.64 28.34) (layer "F.Adhes") (width 0.05) (fill none))
+  (gr_circle (center 345.44 96.52) (end 375.44 96.52) (layer "F.Adhes") (width 0.05) (fill none))
+  (gr_rect (start 404.1 109.22) (end 434.1 106.68) (layer "F.Adhes") (width 0.05) (fill none))
+  (gr_circle (center 101.46 157.34) (end 186.46 157.34) (layer "Edge.Cuts") (width 0.2) (fill none))
+  (gr_rect (start 254 110) (end 424.18 112) (layer "Edge.Cuts") (width 0.2) (fill none))
+  (gr_rect (start 254 53) (end 424.18 55) (layer "Edge.Cuts") (width 0.2) (fill none))
   (gr_rect (start 76.2 104.14) (end 126.2 204.14) (layer "Edge.Cuts") (width 0.2) (fill none))
   (gr_circle (center 101.6 116.84) (end 104.14 116.84) (layer "Margin") (width 0.2) (fill none))
@@
     (effects (font (size 3 3) (thickness 0.375)))
   )
+  (gr_text "H-Bridge (Bottom)" (at 81.28 215.9) (layer "Cmts.User")
+    (effects (font (size 1.5 1.5) (thickness 0.3)) (justify left))
+  )
+  (gr_text "Front" (at 429.26 58.42) (layer "Cmts.User")
+    (effects (font (size 3 3) (thickness 0.375)))
+  )
+  (gr_text "Line Sensors (SEN)" (at 419.1 104.14) (layer "User.5")
+    (effects (font (size 1 1) (thickness 0.15)))
+  )
+  (gr_text "Ultrasonic Sensor" (at 414.02 30.48) (layer "User.5")
+    (effects (font (size 1 1) (thickness 0.15)))
+  )
   (gr_text "SEN4" (at 137.16 99.06) (layer "User.7")
     (effects (font (size 1.5 1.5) (thickness 0.3)) (justify left))
   )
   (gr_text "TT & Encoder R" (at 142.24 180.34) (layer "User.7")
-    (effects (font (size 1.5 1.5) (thickness 0.3)) (justify left))
-  )
-  (gr_text "H-Bridge (Bottom)" (at 81.28 215.9) (layer "User.7")
     (effects (font (size 1.5 1.5) (thickness 0.3)) (justify left))
   )
@@
   )
   (gr_text "Male Connector 2" (at 124.46 152.4 90) (layer "User.9")
-    (effects (font (size 1.5 1.5) (thickness 0.3)))
+    (effects (font (size 1 1) (thickness 0.15)))
   )
   (gr_text "Arduino Nano 33 IoT" (at 101.6 137.16) (layer "User.9")
@@
   )
   (gr_text "Male Connector 1" (at 78.74 152.4 90) (layer "User.9")
-    (effects (font (size 1.5 1.5) (thickness 0.3)))
+    (effects (font (size 1 1) (thickness 0.15)))
   )
   (gr_text "LVL Shift2\n" (at 101.6 193.04) (layer "User.9")
     (effects (font (size 1.5 1.5) (thickness 0.3)))
   )
-  (dimension (type aligned) (layer "Dwgs.User")
-    (pts (xy 16.46 157.34) (xy 186.46 157.34))
-    (height -111.76)
-    (gr_text "170 mm" (at 101.46 43.78) (layer "Dwgs.User")
-      (effects (font (size 1.5 1.5) (thickness 0.3)))
+  (dimension (type aligned) (layer "F.Adhes")
+    (pts (xy 422.91 28.34) (xy 422.91 53.34))
+    (height -13.97)
+    (gr_text "25,0000 mm" (at 435.73 40.84 90) (layer "F.Adhes")
+      (effects (font (size 1 1) (thickness 0.15)))
     )
-    (format (units 3) (units_format 1) (precision 0))
-    (style (thickness 0.2) (arrow_length 1.27) (text_position_mode 0) (extension_height 0.58642) (extension_offset 0.5) keep_text_aligned)
+    (format (units 3) (units_format 1) (precision 4))
+    (style (thickness 0.05) (arrow_length 1.27) (text_position_mode 0) (extension_height 0.58642) (extension_offset 0.5) keep_text_aligned)
+  )
+  (dimension (type aligned) (layer "F.Adhes")
+    (pts (xy 345.44 66.52) (xy 345.44 126.52))
+    (height 40.64)
+    (gr_text "60,0000 mm" (at 303.65 96.52 90) (layer "F.Adhes")
+      (effects (font (size 1 1) (thickness 0.15)))
+    )
+    (format (units 3) (units_format 1) (precision 4))
+    (style (thickness 0.05) (arrow_length 1.27) (text_position_mode 0) (extension_height 0.58642) (extension_offset 0.5) keep_text_aligned)
   )
   (dimension (type aligned) (layer "Edge.Cuts")
@@
   )
   (dimension (type aligned) (layer "Edge.Cuts")
+    (pts (xy 16.46 157.34) (xy 186.46 157.34))
+    (height -111.76)
+    (gr_text "170 mm" (at 101.46 43.78) (layer "Edge.Cuts")
+      (effects (font (size 1.5 1.5) (thickness 0.3)))
+    )
+    (format (units 3) (units_format 1) (precision 0))
+    (style (thickness 0.2) (arrow_length 1.27) (text_position_mode 0) (extension_height 0.58642) (extension_offset 0.5) keep_text_aligned)
+  )
+  (dimension (type aligned) (layer "Edge.Cuts")
     (pts (xy 76.2 104.14) (xy 126.2 104.14))
     (height -5.08)
@@
     (style (thickness 0.2) (arrow_length 1.27) (text_position_mode 0) (extension_height 0.58642) (extension_offset 0.5) keep_text_aligned)
   )
+  (dimension (type aligned) (layer "Edge.Cuts")
+    (pts (xy 254 55) (xy 254 110))
+    (height 15.24)
+    (gr_text "55,0000 mm" (at 236.96 82.5 90) (layer "Edge.Cuts")
+      (effects (font (size 1.5 1.5) (thickness 0.3)))
+    )
+    (format (units 3) (units_format 1) (precision 4))
+    (style (thickness 0.2) (arrow_length 1.27) (text_position_mode 0) (extension_height 0.58642) (extension_offset 0.5) keep_text_aligned)
+  )
