File: KiCAD/Line_Tracking_sch.kicad_sch (KiCad schematic)
At the start: 11 parts

Commit message: Updated schematics and design
Parts:
- gave numbers to parts that had none: 11
Connections:
- net at R2.2, U5.3: now also U6.2 (-)
Other:
- title: (none) -> Line Following Sensor
Changed lines of the file:
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@@
 (kicad_sch (version 20211123) (generator eeschema)
   (paper "A4")
+  (title_block
+    (title "Line Following Sensor")
+    (date "2023-08-06")
+    (rev "v1.0")
+    (comment 2 "EEE3099F")
+    (comment 3 "University of Cape Town")
+    (comment 4 "Friso Vijverberg")
+    (comment 5 "Obtained from:")
+    (comment 6 "https://www.digikey.com/en/products/detail/dfrobot/SEN0017/6588488")
+  )
   (junction (at 140.97 96.52) (diameter 0) (color 0 0 0 0)
   )
@@
   (junction (at 60.96 83.82) (diameter 0) (color 0 0 0 0)
   )
+  (junction (at 68.58 99.06) (diameter 0) (color 0 0 0 0)
+  )
   (junction (at 137.16 52.07) (diameter 0) (color 0 0 0 0)
   )
@@
   )
   (wire (pts (xy 143.51 64.77) (xy 143.51 69.85))
+    (stroke (width 0) (type default) (color 0 0 0 0))
+  )
+  (wire (pts (xy 68.58 99.06) (xy 104.14 99.06))
     (stroke (width 0) (type default) (color 0 0 0 0))
   )
@@
   (symbol (lib_id "power:GND") (at 137.16 69.85 0) (unit 1)
     (in_bom yes) (on_board yes) (fields_autoplaced)
-    (property "Reference" "#PWR?" (id 0) (at 137.16 76.2 0)
+    (property "Reference" "#PWR012" (id 0) (at 137.16 76.2 0)
       (effects (font (size 1.27 1.27)) hide)
     )
@@
   (symbol (lib_id "Sensor_Proximity:ITR8307-S17-TR8") (at 59.69 101.6 0) (unit 1)
     (in_bom yes) (on_board yes) (fields_autoplaced)
-    (property "Reference" "U?" (id 0) (at 59.69 92.71 0))
+    (property "Reference" "U5" (id 0) (at 59.69 92.71 0))
     (property "Value" "ITR8307-S17-TR8" (id 1) (at 59.69 95.25 0)
       (effects (font (size 1.27 1.27)) hide)
@@
   (symbol (lib_id "power:VCC") (at 109.22 85.09 0) (unit 1)
     (in_bom yes) (on_board yes) (fields_autoplaced)
-    (property "Reference" "#PWR?" (id 0) (at 109.22 88.9 0)
+    (property "Reference" "#PWR09" (id 0) (at 109.22 88.9 0)
       (effects (font (size 1.27 1.27)) hide)
     )
@@
   (symbol (lib_id "power:GND") (at 87.63 121.92 0) (unit 1)
     (in_bom yes) (on_board yes) (fields_autoplaced)
-    (property "Reference" "#PWR?" (id 0) (at 87.63 128.27 0)
+    (property "Reference" "#PWR08" (id 0) (at 87.63 128.27 0)
       (effects (font (size 1.27 1.27)) hide)
     )
@@
   (symbol (lib_id "power:VCC") (at 175.26 91.44 0) (unit 1)
     (in_bom yes) (on_board yes) (fields_autoplaced)
-    (property "Reference" "#PWR?" (id 0) (at 175.26 95.25 0)
+    (property "Reference" "#PWR014" (id 0) (at 175.26 95.25 0)
       (effects (font (size 1.27 1.27)) hide)
     )
@@
   (symbol (lib_id "pspice:OPAMP") (at 111.76 96.52 0) (unit 1)
     (in_bom yes) (on_board yes) (fields_autoplaced)
-    (property "Reference" "U?" (id 0) (at 121.92 91.821 0))
+    (property "Reference" "U6" (id 0) (at 121.92 91.821 0))
     (property "Value" "OPAMP" (id 1) (at 121.92 94.361 0))
     (property "Footprint" "" (id 2) (at 111.76 96.52 0)
@@
   (symbol (lib_id "power:VCC") (at 60.96 81.28 0) (unit 1)
     (in_bom yes) (on_board yes) (fields_autoplaced)
-    (property "Reference" "#PWR?" (id 0) (at 60.96 85.09 0)
+    (property "Reference" "#PWR07" (id 0) (at 60.96 85.09 0)
       (effects (font (size 1.27 1.27)) hide)
     )
@@
   (symbol (lib_id "Device:R") (at 140.97 111.76 0) (unit 1)
     (in_bom yes) (on_board yes) (fields_autoplaced)
-    (property "Reference" "R?" (id 0) (at 143.51 110.4899 0)
+    (property "Reference" "R5" (id 0) (at 143.51 110.4899 0)
       (effects (font (size 1.27 1.27)) (justify left))
     )
@@
   (symbol (lib_id "power:VCC") (at 137.16 52.07 0) (unit 1)
     (in_bom yes) (on_board yes) (fields_autoplaced)
-    (property "Reference" "#PWR?" (id 0) (at 137.16 55.88 0)
+    (property "Reference" "#PWR011" (id 0) (at 137.16 55.88 0)
       (effects (font (size 1.27 1.27)) hide)
     )
@@
   (symbol (lib_id "Device:R") (at 50.8 88.9 0) (unit 1)
     (in_bom yes) (on_board yes) (fields_autoplaced)
-    (property "Reference" "R?" (id 0) (at 53.34 87.6299 0)
+    (property "Reference" "R1" (id 0) (at 53.34 87.6299 0)
       (effects (font (size 1.27 1.27)) (justify left))
     )
@@
   (symbol (lib_id "power:GND") (at 109.22 104.14 0) (unit 1)
     (in_bom yes) (on_board yes) (fields_autoplaced)
-    (property "Reference" "#PWR?" (id 0) (at 109.22 110.49 0)
+    (property "Reference" "#PWR010" (id 0) (at 109.22 110.49 0)
       (effects (font (size 1.27 1.27)) hide)
     )
@@
   (symbol (lib_id "Device:LED") (at 140.97 125.73 90) (unit 1)
     (in_bom yes) (on_board yes) (fields_autoplaced)
-    (property "Reference" "D?" (id 0) (at 144.78 126.0474 90)
+    (property "Reference" "D2" (id 0) (at 144.78 126.0474 90)
       (effects (font (size 1.27 1.27)) (justify right))
     )
@@
   (symbol (lib_id "Device:R") (at 68.58 87.63 0) (unit 1)
     (in_bom yes) (on_board yes) (fields_autoplaced)
-    (property "Reference" "R?" (id 0) (at 71.12 86.3599 0)
+    (property "Reference" "R2" (id 0) (at 71.12 86.3599 0)
       (effects (font (size 1.27 1.27)) (justify left))
     )
@@
   (symbol (lib_id "Device:C") (at 143.51 60.96 0) (unit 1)
     (in_bom yes) (on_board yes) (fields_autoplaced)
-    (property "Reference" "C?" (id 0) (at 147.32 59.6899 0)
+    (property "Reference" "C3" (id 0) (at 147.32 59.6899 0)
       (effects (font (size 1.27 1.27)) (justify left))
     )
@@
   (symbol (lib_id "power:GND") (at 140.97 135.89 0) (unit 1)
     (in_bom yes) (on_board yes) (fields_autoplaced)
-    (property "Reference" "#PWR?" (id 0) (at 140.97 142.24 0)
+    (property "Reference" "#PWR013" (id 0) (at 140.97 142.24 0)
       (effects (font (size 1.27 1.27)) hide)
     )
@@
   (symbol (lib_id "Device:C") (at 130.81 60.96 0) (unit 1)
     (in_bom yes) (on_board yes) (fields_autoplaced)
-    (property "Reference" "C?" (id 0) (at 134.62 59.6899 0)
+    (property "Reference" "C2" (id 0) (at 134.62 59.6899 0)
       (effects (font (size 1.27 1.27)) (justify left))
     )
@@
   (symbol (lib_id "power:GND") (at 175.26 104.14 0) (unit 1)
     (in_bom yes) (on_board yes) (fields_autoplaced)
-    (property "Reference" "#PWR?" (id 0) (at 175.26 110.49 0)
+    (property "Reference" "#PWR015" (id 0) (at 175.26 110.49 0)
       (effects (font (size 1.27 1.27)) hide)
     )
@@
   (symbol (lib_id "Device:C") (at 87.63 105.41 0) (unit 1)
     (in_bom yes) (on_board yes) (fields_autoplaced)
-    (property "Reference" "C?" (id 0) (at 91.44 104.1399 0)
+    (property "Reference" "C1" (id 0) (at 91.44 104.1399 0)
       (effects (font (size 1.27 1.27)) (justify left))
     )
@@
   (symbol (lib_id "Device:R") (at 81.28 105.41 0) (unit 1)
     (in_bom yes) (on_board yes) (fields_autoplaced)
-    (property "Reference" "R?" (id 0) (at 83.82 104.1399 0)
+    (property "Reference" "R4" (id 0) (at 83.82 104.1399 0)
       (effects (font (size 1.27 1.27)) (justify left))
     )
@@
   (symbol (lib_id "Device:R") (at 81.28 87.63 0) (unit 1)
     (in_bom yes) (on_board yes) (fields_autoplaced)
-    (property "Reference" "R?" (id 0) (at 83.82 86.3599 0)
-      (effects (font (size 1.27 1.27)) (justify left))
-    )
+    (property "Reference" "R3" (id 0) (at 83.82 86.3599 0)
+      (effects (font (size 1.27 1.27)) (justify left))
+    )

Commit message: Add files via upload
Parts:
- C1: value C -> 10uF
- R1: value R -> 300R
- R2: value R -> 10k
- R3, R4: value R -> 22k
Other:
- moved on the sheet: C1, C2, C3, D2, R1, R2, R3, R4, R5, U5, U6
