File: KiCAD/Motor_Driver_sch.kicad_sch (KiCad schematic)
At the start: 4 parts

Commit message: Updated schematics and design
Parts:
- gave numbers to parts that had none: 4
Connections:
- net D8 renamed D4
Other:
- note added: "En and IN pins set to low before power on"
- note added: "Logic Voltage: 5V"
- note added: "Motor rails connected to Vdd and GND Out 1-4 connected to encoder for each motor respectively"
- note added: "Note: Only the IC is shown here The IC is actually mounted on a module The PINOUT remians the same"
- note added: "Vs - 7.4V input Vss - 5V Logic output Disconnect W1 Jumper"
- note removed: "Motor does not include encoder. Out should go to encoder Place entrire schematic on?"
- title: (none) -> Electromechanical Subsystem
Changed lines of the file:
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@@
 (kicad_sch (version 20211123) (generator eeschema)
   (paper "A4")
+  (title_block
+    (title "Electromechanical Subsystem")
+    (date "2023-08-06")
+    (rev "v1.0")
+    (comment 2 "EEE3099F")
+    (comment 3 "University of Cape Town")
+    (comment 4 "Friso Vijverberg")
+  )
   (junction (at 129.54 104.14) (diameter 0) (color 0 0 0 0)
   )
@@
     (stroke (width 0) (type default) (color 0 0 0 0))
   )
-  (text "IN1 - 4 must have PWM capabilities\n" (at 58.42 82.55 0)
-    (effects (font (size 1.27 1.27)) (justify left bottom))
-  )
-  (text "Motor does not include encoder.\nOut should go to encoder\nPlace entrire schematic on?"
-    (at 166.37 60.96 0)
+  (text "IN1 - 4 must have PWM capabilities\n" (at 74.93 95.25 0)
+    (effects (font (size 1.27 1.27)) (justify left bottom))
+  )
+  (text "En and IN pins set to low before power on\n" (at 74.93 92.71 0)
+    (effects (font (size 1.27 1.27)) (justify left bottom))
+  )
+  (text "Logic Voltage: 5V\n" (at 148.59 86.36 0)
+    (effects (font (size 1.27 1.27)) (justify left bottom))
+  )
+  (text "Vs - 7.4V input\nVss - 5V Logic output\nDisconnect W1 Jumper\n"
+    (at 128.27 58.42 0)
+    (effects (font (size 1.27 1.27)) (justify left bottom))
+  )
+  (text "Motor rails connected to Vdd and GND\nOut 1-4 connected to encoder for each motor respectively\n\n"
+    (at 162.56 69.85 0)
+    (effects (font (size 1.27 1.27)) (justify left bottom))
+  )
+  (text "Note: \nOnly the IC is shown here\nThe IC is actually mounted on a module\nThe PINOUT remians the same"
+    (at 125.73 24.13 0)
     (effects (font (size 1.27 1.27)) (justify left bottom))
   )
@@
     (effects (font (size 1.27 1.27)) (justify right))
   )
-  (hierarchical_label "D8" (shape input) (at 101.6 88.9 180)
+  (hierarchical_label "D4" (shape input) (at 101.6 88.9 180)
     (effects (font (size 1.27 1.27)) (justify right))
   )
@@
   (symbol (lib_id "power:GND") (at 134.62 104.14 0) (unit 1)
     (in_bom yes) (on_board yes) (fields_autoplaced)
-    (property "Reference" "#PWR?" (id 0) (at 134.62 110.49 0)
+    (property "Reference" "#PWR06" (id 0) (at 134.62 110.49 0)
       (effects (font (size 1.27 1.27)) hide)
     )
@@
   (symbol (lib_id "Motor:Motor_DC") (at 170.18 93.98 0) (unit 1)
     (in_bom yes) (on_board yes) (fields_autoplaced)
-    (property "Reference" "M?" (id 0) (at 175.26 95.2499 0)
+    (property "Reference" "M2" (id 0) (at 175.26 95.2499 0)
       (effects (font (size 1.27 1.27)) (justify left))
     )
@@
   (symbol (lib_id "Device:Battery") (at 93.98 58.42 0) (unit 1)
     (in_bom yes) (on_board yes) (fields_autoplaced)
-    (property "Reference" "BT?" (id 0) (at 97.79 56.7689 0)
+    (property "Reference" "BT1" (id 0) (at 97.79 56.7689 0)
       (effects (font (size 1.27 1.27)) (justify left))
     )
@@
   (symbol (lib_id "Motor:Motor_DC") (at 170.18 76.2 0) (unit 1)
     (in_bom yes) (on_board yes) (fields_autoplaced)
-    (property "Reference" "M?" (id 0) (at 175.26 77.4699 0)
+    (property "Reference" "M1" (id 0) (at 175.26 77.4699 0)
       (effects (font (size 1.27 1.27)) (justify left))
     )
@@
   (symbol (lib_id "power:GND") (at 93.98 66.04 0) (unit 1)
     (in_bom yes) (on_board yes) (fields_autoplaced)
-    (property "Reference" "#PWR?" (id 0) (at 93.98 72.39 0)
+    (property "Reference" "#PWR05" (id 0) (at 93.98 72.39 0)
       (effects (font (size 1.27 1.27)) hide)
     )
@@
   (symbol (lib_id "Driver_Motor:L298N") (at 134.62 86.36 0) (unit 1)
     (in_bom yes) (on_board yes) (fields_autoplaced)
-    (property "Reference" "U?" (id 0) (at 139.1794 66.04 0)
-      (effects (font (size 1.27 1.27)) (justify left))
-    )
+    (property "Reference" "U4" (id 0) (at 139.1794 66.04 0)
+      (effects (font (size 1.27 1.27)) (justify left))
+    )

Commit message: Add files via upload
Connections:
- net D10/PWM renamed IN4
- net D4 renamed EN
- net D5/PWM renamed IN1
- net D6/PWM renamed IN2
- net D9/PWM renamed IN3
Other:
- moved on the sheet: BT1, M1, M2, U4
